Commit message: Update djidrone.urdf

File: urdf/dji drone.urdf (robot description, URDF)
Before this commit: robot dji drone, 5 links, 4 joints
Links:
- link Link_1: geometry collision mesh filename=package://djidrone/meshes/Link_1.STL; visual mesh filename=package://djidrone/meshes/Link_1.STL
- link Link_2: geometry collision mesh filename=package://djidrone/meshes/Link_2.STL; visual mesh filename=package://djidrone/meshes/Link_2.STL
- link Link_3: geometry collision mesh filename=package://djidrone/meshes/Link_3.STL; visual mesh filename=package://djidrone/meshes/Link_3.STL
- link Link_4: geometry collision mesh filename=package://djidrone/meshes/Link_4.STL; visual mesh filename=package://djidrone/meshes/Link_4.STL
- link base_link: geometry collision mesh filename=package://djidrone/meshes/base_link.STL; visual mesh filename=package://djidrone/meshes/base_link.STL
